File: MS-shema_1.0.sch (KiCad schematic (older format))
At the start: 49 parts, among them M1 Motor Levi, M2 Motor Desni, Q1 Q_NPN_CBE, Q2 Q_PMOS_GSD, SW1 SWITCH_INV

Commit message: Dodani footprinti ter PCB
Dodana je končna shema, narisani so footprinti komponent in PCB design
(opomba: Glavni PCB design je pod MS-shema_1.0.pcb. Ostale datoteke so
le rezultat vmesnega shranjevanja, ampak si jih žal ne upam zbrisati,
ker nisem popolnoma prepričan katere datoteke Ki-Cad potrebuje in katere
ne (je že pozno in ne bi rad vsega ponovno delal :) )
Parts:
- removed SH1: Shifter, symbol Shifter
- added Q3, Q4: BSS138, TO_SOT_Packages_SMD:SOT-23_Handsoldering, symbol BSS138
- added R23, R24, R25, R26: 10K, Resistors_SMD:R_1210_HandSoldering, symbol R
- BT1: footprint (none) -> Robot:BatteryHolder9V
- BT2: footprint (none) -> Robot:RN42
- C1: footprint (none) -> Capacitors_SMD:CP_Elec_5x4.5
- DRV1: footprint (none) -> Robot:TB6612FNG
- LS1, LS10, LS11, LS12, LS13, LS14, LS15, LS2, LS3, LS4, LS5, LS6, LS7, LS8, LS9: footprint (none) -> Robot:QRE1113; symbol QRE1113 -> QRE1113-RESCUE-MS-shema_1.0
- M1, M2: footprint (none) -> Robot:Encoder
- MUX1: footprint (none) -> Robot:CD74HC4067
- Q1: footprint (none) -> TO_SOT_Packages_THT:TO-3PB__Vertical
- Q2: footprint (none) -> TO_SOT_Packages_SMD:SOT-23_Handsoldering
- R1, R10, R11, R12, R13, R14, R15, R16, R17, R18, R19, R2, R20, R21, R22, R3, R4, R5, R6, R7, R8, R9: footprint (none) -> Resistors_SMD:R_1210_HandSoldering
- SW1: footprint (none) -> Robot:switch
- UC1: footprint (none) -> Robot:ArduinoMicro
Connections:
- net +3V3: now also Q3.1 (G), Q4.1 (G), R23.2, R24.2
- net +5V: now also R25.2, R26.2
- net RX: now also Q4.3 (D), R26.1
- net TX: now also Q3.3 (D), R25.1
- net at BT2.13 (UART_RX): now also Q4.2 (S), R24.1
- net at BT2.14 (UART_TX): now also Q3.2 (S), R23.1
- no-connect marks 39 -> 35
Other:
- moved on the sheet: BT1, BT2, C1, Q2, R10, R11, R9, SW1
